Commit message: working s100

File: urdf/arm.urdf.xacro (robot description, xacro)
@@ -1,128 +1,231 @@
 <?xml version="1.0"?>
-<robot name="articulate_2d" xmlns:xacro="http://www.ros.org/wiki/xacro">
-  <!-- BASE LINK — this is the root, fixed to world by Ignition automatically -->
-  <link name="base_link">
-    <visual>
-      <origin xyz="0 0 0.05" rpy="0 0 0"/>
-      <geometry>
-        <box size="0.3 0.3 0.1"/>
-      </geometry>
-      <material name="blue">
-        <color rgba="0 0 1 1"/>
-      </material>
-    </visual>
-    <collision>
-      <origin xyz="0 0 0.05" rpy="0 0 0"/>
-      <geometry>
-        <box size="0.3 0.3 0.1"/>
-      </geometry>
-    </collision>
-    <inertial>
-      <origin xyz="0 0 0.05" rpy="0 0 0"/>
-      <mass value="2.0"/>
-      <inertia ixx="0.1" iyy="0.1" izz="0.1"
-               ixy="0.0" ixz="0.0" iyz="0.0"/>
-    </inertial>
-  </link>
-  <!-- LINK 1 -->
-  <link name="link1">
-    <visual>
-      <origin xyz="0 0 0.5" rpy="0 0 0"/>
-      <geometry>
-        <cylinder length="1.0" radius="0.06"/>
-      </geometry>
-      <material name="green">
-        <color rgba="0 1 0 1"/>
-      </material>
-    </visual>
-    <collision>
-      <origin xyz="0 0 0.5" rpy="0 0 0"/>
-      <geometry>
-        <cylinder length="1.0" radius="0.06"/>
-      </geometry>
-    </collision>
-    <inertial>
-      <origin xyz="0 0 0.5" rpy="0 0 0"/>
-      <mass value="1.5"/>
-      <inertia ixx="0.1375" iyy="0.1375" izz="0.0027"
-               ixy="0.0" ixz="0.0" iyz="0.0"/>
-    </inertial>
-  </link>
-  <!-- LINK 2 -->
-  <link name="link2">
-    <visual>
-      <origin xyz="0 0 0.5" rpy="0 0 0"/>
-      <geometry>
-        <cylinder length="1.0" radius="0.05"/>
-      </geometry>
-      <material name="red">
-        <color rgba="1 0 0 1"/>
-      </material>
-    </visual>
-    <collision>
-      <origin xyz="0 0 0.5" rpy="0 0 0"/>
-      <geometry>
-        <cylinder length="1.0" radius="0.05"/>
-      </geometry>
-    </collision>
-    <inertial>
-      <origin xyz="0 0 0.5" rpy="0 0 0"/>
+<robot name="so_arm100" xmlns:xacro="http://www.ros.org/wiki/xacro">
+  <!-- WORLD -->
+  <link name="world"/>
+  <!-- MATERIALS -->
+  <material name="3d_printed">
+    <color rgba="1.0 0.82 0.12 1.0"/>
+  </material>
+  <material name="sts3215">
+    <color rgba="0.1 0.1 0.1 1.0"/>
+  </material>
+  <!-- BASE -->
+  <link name="base">
+    <inertial>
       <mass value="1.0"/>
-      <inertia ixx="0.0854" iyy="0.0854" izz="0.00125"
-               ixy="0.0" ixz="0.0" iyz="0.0"/>
-    </inertial>
-  </link>
-  <!-- JOINT 1: base_link → link1
-       base visual is 0.1 tall centered at 0.05, so top surface is at z=0.1 -->
-  <joint name="joint1" type="revolute">
-    <parent link="base_link"/>
-    <child link="link1"/>
-    <origin xyz="0 0 0.1" rpy="0 0 0"/>
+      <inertia ixx="0.01" iyy="0.01" izz="0.01"
+               ixy="0" ixz="0" iyz="0"/>
+    </inertial>
+    <visual>
+      <geometry>
+        <mesh filename="/home/rafi/Documents/Robotics/articulate2d_ws/src/articulate_2d/meshes/Base.stl"/>
+      </geometry>
+      <material name="3d_printed"/>
+    </visual>
+    <visual>
+      <geometry>
+        <mesh filename="/home/rafi/Documents/Robotics/articulate2d_ws/src/articulate_2d/meshes/Base_Motor.stl"/>
+      </geometry>
+      <material name="sts3215"/>
+    </visual>
+    <collision>
+      <geometry>
+        <mesh filename="/home/rafi/Documents/Robotics/articulate2d_ws/src/articulate_2d/meshes/Base.stl"/>
+      </geometry>
+    </collision>
+  </link>
+  <!-- FIX BASE -->
+  <joint name="fixed_base" type="fixed">
+    <parent link="world"/>
+    <child link="base"/>
+  </joint>
+  <!-- SHOULDER -->
+  <link name="shoulder">
+    <inertial>
+      <mass value="0.12"/>
+      <inertia ixx="0.00006" iyy="0.00006" izz="0.00003"
+               ixy="0" ixz="0" iyz="0"/>
+    </inertial>
+    <visual>
+      <geometry>
+        <mesh filename="/home/rafi/Documents/Robotics/articulate2d_ws/src/articulate_2d/meshes/Rotation_Pitch.stl"/>
+      </geometry>
+      <material name="3d_printed"/>
+    </visual>
+    <collision>
+      <geometry>
+        <mesh filename="/home/rafi/Documents/Robotics/articulate2d_ws/src/articulate_2d/meshes/Rotation_Pitch.stl"/>
+      </geometry>
+    </collision>
+  </link>
+  <joint name="shoulder_pan" type="revolute">
+    <parent link="base"/>
+    <child link="shoulder"/>
+    <origin xyz="0 -0.0452 0.0165" rpy="1.57 0 0"/>
+    <axis xyz="0 1 0"/>
+    <limit lower="-2" upper="2" effort="35" velocity="1"/>
+  </joint>
+  <!-- UPPER ARM -->
+  <link name="upper_arm">
+    <inertial>
+      <mass value="0.16"/>
+      <inertia ixx="0.0002" iyy="0.00017" izz="0.00007"
+               ixy="0" ixz="0" iyz="0"/>
+    </inertial>
+    <visual>
+      <geometry>
+        <mesh filename="/home/rafi/Documents/Robotics/articulate2d_ws/src/articulate_2d/meshes/Upper_Arm.stl"/>
+      </geometry>
+      <material name="3d_printed"/>
+    </visual>
+    <collision>
+      <geometry>
+        <mesh filename="/home/rafi/Documents/Robotics/articulate2d_ws/src/articulate_2d/meshes/Upper_Arm.stl"/>
+      </geometry>
+    </collision>
+  </link>
+  <joint name="shoulder_lift" type="revolute">
+    <parent link="shoulder"/>
+    <child link="upper_arm"/>
+    <origin xyz="0 0.1025 0.0306" rpy="-1.8 0 0"/>
+    <axis xyz="1 0 0"/>
+    <limit lower="0" upper="3.5" effort="35" velocity="1"/>
+  </joint>
+  <!-- LOWER ARM -->
+  <link name="lower_arm">
+    <inertial>
+      <mass value="0.15"/>
+      <inertia ixx="0.00013" iyy="0.00010" izz="0.00005"
+               ixy="0" ixz="0" iyz="0"/>
+    </inertial>
+    <visual>
+      <geometry>
+        <mesh filename="/home/rafi/Documents/Robotics/articulate2d_ws/src/articulate_2d/meshes/Lower_Arm.stl"/>
+      </geometry>
+      <material name="3d_printed"/>
+    </visual>
+    <collision>
+      <geometry>
+        <mesh filename="/home/rafi/Documents/Robotics/articulate2d_ws/src/articulate_2d/meshes/Lower_Arm.stl"/>
+      </geometry>
+    </collision>
+  </link>
+  <joint name="elbow_flex" type="revolute">
+    <parent link="upper_arm"/>
+    <child link="lower_arm"/>
+    <origin xyz="0 0.1125 0.028" rpy="1.57 0 0"/>
+    <axis xyz="1 0 0"/>
+    <limit lower="-3.14" upper="0" effort="35" velocity="1"/>
+  </joint>
+  <!-- WRIST -->
+  <link name="wrist">
+    <inertial>
+      <mass value="0.07"/>
+      <inertia ixx="0.00003" iyy="0.00002" izz="0.00002"
+               ixy="0" ixz="0" iyz="0"/>
+    </inertial>
+    <visual>
+      <geometry>
+        <mesh filename="/home/rafi/Documents/Robotics/articulate2d_ws/src/articulate_2d/meshes/Wrist_Pitch_Roll.stl"/>
+      </geometry>
+      <material name="3d_printed"/>
+    </visual>
+    <collision>
+      <geometry>
+        <mesh filename="/home/rafi/Documents/Robotics/articulate2d_ws/src/articulate_2d/meshes/Wrist_Pitch_Roll.stl"/>
+      </geometry>
+    </collision>
+  </link>
+  <joint name="wrist_flex" type="revolute">
+    <parent link="lower_arm"/>
+    <child link="wrist"/>
+    <origin xyz="0 0.0052 0.1349" rpy="-1 0 0"/>
+    <axis xyz="1 0 0"/>
+    <limit lower="-2.5" upper="1.2" effort="35" velocity="1"/>
+  </joint>
+  <!-- GRIPPER -->
+  <link name="gripper">
+    <inertial>
+      <mass value="0.09"/>
+      <inertia ixx="0.00005" iyy="0.00004" izz="0.00003"
+               ixy="0" ixz="0" iyz="0"/>
+    </inertial>
+    <visual>
+      <geometry>
+        <mesh filename="/home/rafi/Documents/Robotics/articulate2d_ws/src/articulate_2d/meshes/Fixed_Jaw.stl"/>
+      </geometry>
+      <material name="3d_printed"/>
+    </visual>
+  </link>
+  <joint name="wrist_roll" type="revolute">
+    <parent link="wrist"/>
+    <child link="gripper"/>
+    <origin xyz="0 -0.0601 0" rpy="0 1.57 0"/>
+    <axis xyz="0 1 0"/>
+    <limit lower="-3.14" upper="3.14" effort="35" velocity="1"/>
+  </joint>
+  <!-- JAW -->
+  <link name="jaw">
+    <inertial>
+      <mass value="0.02"/>
+      <inertia ixx="1e-05" iyy="1e-05" izz="1e-06"
+               ixy="0" ixz="0" iyz="0"/>
+    </inertial>
+    <visual>
+      <geometry>
+        <mesh filename="/home/rafi/Documents/Robotics/articulate2d_ws/src/articulate_2d/meshes/Moving_Jaw.stl"/>
+      </geometry>
+      <material name="3d_printed"/>
+    </visual>
+  </link>
+  <joint name="gripper_joint" type="revolute">
+    <parent link="gripper"/>
+    <child link="jaw"/>
+    <origin xyz="-0.02 -0.02 0" rpy="0 3.14 0"/>
     <axis xyz="0 0 1"/>
-    <limit effort="10" velocity="1.0" lower="-3.14" upper="3.14"/>
-    <dynamics damping="0.1" friction="0.1"/>
-  </joint>
-  <!-- JOINT 2: link1 → link2
-       link1 cylinder is 1.0m long, so top is at z=1.0 in link1 frame -->
-  <joint name="joint2" type="revolute">
-    <parent link="link1"/>
-    <child link="link2"/>
-    <origin xyz="0 0 1.0" rpy="0 0 0"/>
-    <axis xyz="0 0 1"/>
-    <limit effort="10" velocity="1.0" lower="-3.14" upper="3.14"/>
-    <dynamics damping="0.1" friction="0.1"/>
-  </joint>
-  <!-- ROS2 CONTROL — Fortress plugin -->
+    <limit lower="-0.2" upper="2.0" effort="35" velocity="1"/>
+  </joint>
+  <!-- ROS2 CONTROL -->
   <ros2_control name="IgnitionSystem" type="system">
     <hardware>
-      <plugin>ign_ros2_control/IgnitionSystem</plugin>
+      <plugin>gz_ros2_control/GazeboSimSystem</plugin>
     </hardware>
-    <joint name="joint1">
-      <command_interface name="position">
-        <param name="min">-3.14</param>
-        <param name="max">3.14</param>
-      </command_interface>
-      <state_interface name="position"/>
-      <state_interface name="velocity"/>
-    </joint>
-    <joint name="joint2">
-      <command_interface name="position">
-        <param name="min">-3.14</param>
-        <param name="max">3.14</param>
-      </command_interface>
+    <joint name="shoulder_pan">
+      <command_interface name="position"/>
+      <state_interface name="position"/>
+      <state_interface name="velocity"/>
+    </joint>
+    <joint name="shoulder_lift">
+      <command_interface name="position"/>
+      <state_interface name="position"/>
+      <state_interface name="velocity"/>
+    </joint>
+    <joint name="elbow_flex">
+      <command_interface name="position"/>
+      <state_interface name="position"/>
+      <state_interface name="velocity"/>
+    </joint>
+    <joint name="wrist_flex">
+      <command_interface name="position"/>
+      <state_interface name="position"/>
+      <state_interface name="velocity"/>
+    </joint>
+    <joint name="wrist_roll">
+      <command_interface name="position"/>
+      <state_interface name="position"/>
+      <state_interface name="velocity"/>
+    </joint>
+    <joint name="gripper_joint">
+      <command_interface name="position"/>
       <state_interface name="position"/>
       <state_interface name="velocity"/>
     </joint>
   </ros2_control>
-  <!-- GAZEBO FORTRESS PLUGIN -->
+  <!-- GAZEBO PLUGIN -->
   <gazebo>
-    <plugin filename="ign_ros2_control-system"
-            name="ign_ros2_control::IgnitionROS2ControlPlugin">
+    <plugin filename="gz_ros2_control-system"
+        name="gz_ros2_control::GazeboSimROS2ControlPlugin">
       <parameters>/home/rafi/Documents/Robotics/articulate2d_ws/src/articulate_2d/config/controllers.yaml</parameters>
     </plugin>
   </gazebo>
-  <!-- Make base_link fixed to world in Ignition -->
-  <gazebo reference="base_link">
-    <static>false</static>
-  </gazebo>
 </robot>

Commit message: latest working version

File: urdf/arm.urdf.xacro (robot description, xacro)
@@ -19,11 +19,11 @@
     <visual>
       <geometry>
-        <mesh filename="/home/rafi/Documents/Robotics/articulate2d_ws/src/articulate_2d/meshes/Base.stl"/>
-      </geometry>
-      <material name="3d_printed"/>
-    </visual>
-    <visual>
-      <geometry>
-        <mesh filename="/home/rafi/Documents/Robotics/articulate2d_ws/src/articulate_2d/meshes/Base_Motor.stl"/>
+        <mesh filename="package://articulate_2d/meshes/Base.stl"/>
+      </geometry>
+      <material name="3d_printed"/>
+    </visual>
+    <visual>
+      <geometry>
+        <mesh filename="package://articulate_2d/meshes/Base_Motor.stl"/>
       </geometry>
       <material name="sts3215"/>
@@ -31,5 +31,5 @@
     <collision>
       <geometry>
-        <mesh filename="/home/rafi/Documents/Robotics/articulate2d_ws/src/articulate_2d/meshes/Base.stl"/>
+        <mesh filename="package://articulate_2d/meshes/Base.stl"/>
       </geometry>
     </collision>
@@ -49,11 +49,11 @@
     <visual>
       <geometry>
-        <mesh filename="/home/rafi/Documents/Robotics/articulate2d_ws/src/articulate_2d/meshes/Rotation_Pitch.stl"/>
-      </geometry>
-      <material name="3d_printed"/>
-    </visual>
-    <collision>
-      <geometry>
-        <mesh filename="/home/rafi/Documents/Robotics/articulate2d_ws/src/articulate_2d/meshes/Rotation_Pitch.stl"/>
+        <mesh filename="package://articulate_2d/meshes/Rotation_Pitch.stl"/>
+      </geometry>
+      <material name="3d_printed"/>
+    </visual>
+    <collision>
+      <geometry>
+        <mesh filename="package://articulate_2d/meshes/Rotation_Pitch.stl"/>
       </geometry>
     </collision>
@@ -75,11 +75,11 @@
     <visual>
       <geometry>
-        <mesh filename="/home/rafi/Documents/Robotics/articulate2d_ws/src/articulate_2d/meshes/Upper_Arm.stl"/>
-      </geometry>
-      <material name="3d_printed"/>
-    </visual>
-    <collision>
-      <geometry>
-        <mesh filename="/home/rafi/Documents/Robotics/articulate2d_ws/src/articulate_2d/meshes/Upper_Arm.stl"/>
+        <mesh filename="package://articulate_2d/meshes/Upper_Arm.stl"/>
+      </geometry>
+      <material name="3d_printed"/>
+    </visual>
+    <collision>
+      <geometry>
+        <mesh filename="package://articulate_2d/meshes/Upper_Arm.stl"/>
       </geometry>
     </collision>
@@ -101,11 +101,11 @@
     <visual>
       <geometry>
-        <mesh filename="/home/rafi/Documents/Robotics/articulate2d_ws/src/articulate_2d/meshes/Lower_Arm.stl"/>
-      </geometry>
-      <material name="3d_printed"/>
-    </visual>
-    <collision>
-      <geometry>
-        <mesh filename="/home/rafi/Documents/Robotics/articulate2d_ws/src/articulate_2d/meshes/Lower_Arm.stl"/>
+        <mesh filename="package://articulate_2d/meshes/Lower_Arm.stl"/>
+      </geometry>
+      <material name="3d_printed"/>
+    </visual>
+    <collision>
+      <geometry>
+        <mesh filename="package://articulate_2d/meshes/Lower_Arm.stl"/>
       </geometry>
     </collision>
@@ -127,11 +127,11 @@
     <visual>
       <geometry>
-        <mesh filename="/home/rafi/Documents/Robotics/articulate2d_ws/src/articulate_2d/meshes/Wrist_Pitch_Roll.stl"/>
-      </geometry>
-      <material name="3d_printed"/>
-    </visual>
-    <collision>
-      <geometry>
-        <mesh filename="/home/rafi/Documents/Robotics/articulate2d_ws/src/articulate_2d/meshes/Wrist_Pitch_Roll.stl"/>
+        <mesh filename="package://articulate_2d/meshes/Wrist_Pitch_Roll.stl"/>
+      </geometry>
+      <material name="3d_printed"/>
+    </visual>
+    <collision>
+      <geometry>
+        <mesh filename="package://articulate_2d/meshes/Wrist_Pitch_Roll.stl"/>
       </geometry>
     </collision>
@@ -153,5 +153,5 @@
     <visual>
       <geometry>
-        <mesh filename="/home/rafi/Documents/Robotics/articulate2d_ws/src/articulate_2d/meshes/Fixed_Jaw.stl"/>
+        <mesh filename="package://articulate_2d/meshes/Fixed_Jaw.stl"/>
       </geometry>
       <material name="3d_printed"/>
@@ -174,5 +174,5 @@
     <visual>
       <geometry>
-        <mesh filename="/home/rafi/Documents/Robotics/articulate2d_ws/src/articulate_2d/meshes/Moving_Jaw.stl"/>
+        <mesh filename="package://articulate_2d/meshes/Moving_Jaw.stl"/>
       </geometry>
       <material name="3d_printed"/>
@@ -187,5 +187,9 @@
   </joint>
   <!-- ROS2 CONTROL -->
-  <ros2_control name="IgnitionSystem" type="system">
+  <!-- <ros2_control name="IgnitionSystem" type="system">
+    <hardware>
+      <plugin>ign_ros2_control/IgnitionSystem</plugin>
+    </hardware> -->
+  <ros2_control name="GazeboSystem" type="system">
     <hardware>
       <plugin>gz_ros2_control/GazeboSimSystem</plugin>
@@ -228,4 +232,8 @@
       <parameters>/home/rafi/Documents/Robotics/articulate2d_ws/src/articulate_2d/config/controllers.yaml</parameters>
     </plugin>
+<!--
+    <plugin filename="ign_ros2_control-system" name="ign_ros2_control::IgnitionROS2ControlPlugin">
+      <parameters>/home/rafi/Documents/Robotics/articulate2d_ws/src/articulate_2d/config/controllers.yaml</parameters>
+    </plugin> -->
   </gazebo>
 </robot>
